Commit message: 修改了urdf，不再使用与真实机械结构不符的floating类型关节

File: src/rmcv_bringup/urdf/rm_gimbal.urdf.xacro (robot description, xacro)
@@ -2,15 +2,24 @@
 <robot name="rm_gimbal"
   xmlns:xacro="http://ros.org/wiki/xacro">
-  <xacro:arg name="xyz" default="0.10 0 0.05" />
-  <xacro:arg name="rpy" default="0 0 0" />
+  <xacro:arg name="pitch2cam_xyz" default="0.10 0 0.05" />
+  <xacro:arg name="pitch2cam_rpy" default="0 0 0" />
+  <xacro:arg name="yaw2pitch_xyz" default="0.0 0.0 0.0" />
   <link name="odom" />
-  <link name="gimbal_link" />
-  <joint name="gimbal_joint" type="floating">
+  <link name="yaw_link" />
+  <joint name="yaw_joint" type="continuous">
     <parent link="odom" />
-    <child link="gimbal_link" />
+    <child link="yaw_link" />
+    <axis xyz="0 0 1" />
+  </joint>
+  <link name="pitch_link" />
+  <joint name="pitch_joint" type="continuous">
+    <parent link="yaw_link" />
+    <child link="pitch_link" />
+    <origin xyz="$(arg yaw2pitch_xyz)" />
+    <axis xyz="0 1 0" />
   </joint>
   <link name="camera_link" />
   <joint name="camera_joint" type="fixed">
-    <origin xyz="$(arg xyz)" rpy="$(arg rpy)" />
+    <origin xyz="$(arg pitch2cam_xyz)" rpy="$(arg pitch2cam_rpy)" />
     <parent link="gimbal_link" />
     <child link="camera_link" />

Commit message: fix:替换掉了urdf里不应该存在的gimbal_link

File: src/rmcv_bringup/urdf/rm_gimbal.urdf.xacro (robot description, xacro)
@@ -22,5 +22,5 @@
   <joint name="camera_joint" type="fixed">
     <origin xyz="$(arg pitch2cam_xyz)" rpy="$(arg pitch2cam_rpy)" />
-    <parent link="gimbal_link" />
+    <parent link="pitch_link" />
     <child link="camera_link" />
     <axis xyz="0 0 0" />
